File: PCB/macpad.kicad_pcb (KiCad board)
At the start: 2 copper layers, 42.7 x 63.3 mm, 7 parts, among them SW1 SW_Push, SW2 SW_Push, SW3 SW_Push, SW4 SW_Push, U1 XIAO-RP2040-DIP

Commit message: Add files via upload
Parts:
- added D3: SK6812, LED_SMD:LED_SK6812_PLCC4_5.0x5.0mm_P3.2mm, F.Cu at (84.6, 33.6)
- moved D2 1.20 mm to (84.6, 39.6)
Connections:
- D2 pad 1: unconnected-(D2-VSS-Pad1) -> Net-(D2-VSS)
Routing:
- net Net-(D2-VSS): track 0.00 -> 6.06 mm
- net +5V: track 43.1 -> 46.3 mm
- net GND: track 104.1 -> 105.6 mm
